File: apple_night_light.sch (EAGLE design)
At the start: 42 parts, among them U2 INA219AIDCNR, U3 ATSHA204-TSU, Y1 16MHZ

Commit message: final changes before order, reversing tx/rx for ftdi, reset pin on SPI
Connections:
- removed net N$22: C6.2, MP.PC6(/RESET), R4.1
- removed net N$46: AOUT.1, C1.2, C2.-, C3.-, C4.2, C5.2, C7.2, DOUT.1, JP1.CTS, JP1.GND, JP2.GND, LED1.GREEN_C, LED10.GREEN_C, LED11.GREEN_C, LED12.GREEN_C, LED2.GREEN_C, LED3.GREEN_C, LED4.GREEN_C, LED5.GREEN_C, LED6.GREEN_C, LED7.GREEN_C, LED8.GREEN_C, LED9.GREEN_C, MP.AGND, MP.GND@1, MP.GND@2, NRF.1, R1.1, SPI.6, U$1.GND, U$3.GND@1, U$3.GND@2, U$3.IR-@1, U$3.IR-@2, U1.GND, U2.GND, USBOUT.GND, Y1.2
- new net RESET: C6.2, MP.PC6(/RESET), R4.1, SPI.5
- net CSN: no longer SPI.5
- net GND: now also AOUT.1, C1.2, C2.-, C3.-, C4.2, C5.2, C7.2, DOUT.1, JP1.CTS, JP1.GND, JP2.GND, LED1.GREEN_C, LED10.GREEN_C, LED11.GREEN_C, LED12.GREEN_C, LED2.GREEN_C, LED3.GREEN_C, LED4.GREEN_C, LED5.GREEN_C, LED6.GREEN_C, LED7.GREEN_C, LED8.GREEN_C, LED9.GREEN_C, MP.AGND, MP.GND@1, MP.GND@2, NRF.1, R1.1, SPI.6, U$1.GND, U$3.GND@1, U$3.GND@2, U$3.IR-@1, U$3.IR-@2, U1.GND, U2.GND, USBOUT.GND, Y1.2
- net RXI: now also JP1.RXI; no longer JP1.TXO
- net TXO: now also JP1.TXO; no longer JP1.RXI
Other:
- note removed: "Why it TX/RX reversed on pro mini schematic?"

Commit message: fixing issue with grounding VCNL IR emmiter, causes blow out of emmiter :x
Connections:
- net GND: no longer U$3.IR-@1, U$3.IR-@2
Changed lines of the file:
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@@
 <junction x="-76.2" y="12.7"/>
 <pinref part="GND4" gate="1" pin="GND"/>
-<junction x="-76.2" y="17.78"/>
-<pinref part="U$3" gate="G$1" pin="IR-@2"/>
-<wire x1="-81.28" y1="27.94" x2="-76.2" y2="27.94" width="0.1524" layer="91"/>
-<wire x1="-76.2" y1="27.94" x2="-76.2" y2="22.86" width="0.1524" layer="91"/>
-<pinref part="U$3" gate="G$1" pin="IR-@1"/>
-<wire x1="-76.2" y1="22.86" x2="-76.2" y2="17.78" width="0.1524" layer="91"/>
-<wire x1="-81.28" y1="22.86" x2="-76.2" y2="22.86" width="0.1524" layer="91"/>
-<junction x="-76.2" y="22.86"/>
-<junction x="-76.2" y="27.94"/>
 </segment>
 <segment>
